Commit message: Add colors for robot
This commit tries to add color to my_robot. This is done by
both update the URDF file to refrect the real color in rViz,
as well as update the gazebo color.

This also removes any references to the robot in my_world,
which made the color disappear, as well as add a simple script
to spawn the robot in the middle.

File: my_robot/urdf/my_robot.xacro (robot description, xacro)
@@ -31,4 +31,7 @@
         <box size=".4 .2 .1"/>
       </geometry>
+      <material name='blue'>
+        <color rgba="0.0 0.0 1.0 1.0"/>
+      </material>
     </visual>
     <collision name='back_caster_collision'>
@@ -75,4 +78,7 @@
     </collision>
     <visual name='left_wheel_visual'>
+      <material name='green'>
+        <color rgba="0.0 1.0 0.0 1.0"/>
+      </material>
       <origin xyz="0 0 0" rpy="0 1.5707 1.5707"/>
       <geometry>
@@ -102,4 +108,7 @@
         <cylinder radius="0.1" length="0.05"/>
       </geometry>
+      <material name='green'>
+        <color rgba="0.0 1.0 0.0 1.0"/>
+      </material>
     </visual>
   </link>
@@ -143,4 +152,7 @@
         <box size="0.05 0.05 0.05"/>
       </geometry>
+      <material name='red'>
+        <color rgba="1.0 0.0 0.0 1.0"/>
+      </material>
     </visual>
   </link>

Commit message: Use RGBD camera
To prepare for mapping the environment using
RTAB SLAM, this commit changes the robot current
camera to be a RGBD camera with depth perception.

File: my_robot/urdf/my_robot.xacro (robot description, xacro)
@@ -163,4 +163,11 @@
     <axis xyz="0 1 0" rpy="0 0 0"/>
   </joint>
+  <link name="camera_link_optical">
+  </link>
+  <joint name="camera_optical_joint" type="fixed">
+    <origin xyz="0 0 0" rpy="-1.5707 0 -1.5707"/>
+    <parent link="camera"/>
+    <child link="camera_link_optical"/>
+  </joint>
   <link name='hokuyo'>
     <inertial>
